File: CheeseUnua.kicad_pcb (KiCad board)
At the start: 2 copper layers, 96.5 x 63.5 mm, 63 parts, among them J1 Jack-DC, J2 Battery, J3 Conn_01x05, J4 Conn_01x03, J5 Conn_01x06, J6 AE-AQM0802, J7 CN2, J8 CN1, Q1 2SJ681, Q2 2SK2796L, SW1 SW_SPDT, SW2 SW_SPST, SW3 SW_DPST_x2, U1 R-78E3.3-0.5, U2 SLA7073MPRT, U3 7SEGMENT_CA, U4 NJM2742D, U5 NJU7072D

Commit message: Step up to version 2
Parts:
- removed SW1: SW_SPDT, Pin_Headers:Pin_Header_Straight_1x03_Pitch2.54mm
- added JP1: Jumper_3_Bridged12, Pin_Headers:Pin_Header_Straight_1x03_Pitch2.54mm, F.Cu at (94.5, 73.7)
- J5: footprint Connectors_JST:JST_PH_B6B-PH-K_06x2.00mm_Straight -> Connectors_JST:JST_XH_S06B-XH-A_06x2.50mm_Angled
- R1, R10, R11, R12, R13, R14, R15, R16, R17, R18, R19, R2, R20, R21, R22, R23, R25, R26, R3, R4, R5, R6, R7, R8, R9: footprint Resistors_THT:R_Axial_DIN0204_L3.6mm_D1.6mm_P5.08mm_Horizontal -> Resistors_THT:R_Axial_DIN0204_L3.6mm_D1.6mm_P7.62mm_Horizontal
- R24: footprint Resistors_THT:R_Axial_DIN0204_L3.6mm_D1.6mm_P5.08mm_Horizontal -> Resistors_THT:R_Axial_DIN0207_L6.3mm_D2.5mm_P10.16mm_Horizontal
- moved SW3 26.5 mm to (135.1, 113.5), turned to 0 degrees
- moved R10 26.2 mm to (133.3, 109.2)
- moved R11 26.2 mm to (133.3, 106.7)
- moved LS1 24.2 mm to (152.0, 95.7)
- moved J3 22.2 mm to (165.1, 111.4)
- moved U3 22.0 mm to (154.9, 117.1)
- moved R5 8.02 mm to (117.9, 68.6), turned to 180 degrees
- moved D3 4.94 mm to (166.1, 105.4), turned to 180 degrees
- moved R9 4.19 mm to (117.9, 71.6), turned to 180 degrees
- moved R8 3.33 mm to (105.7, 99.1)
- moved R2 2.84 mm to (105.7, 89.4)
- moved R7 2.80 mm to (105.7, 96.0)
- moved R3 1.69 mm to (100.6, 122.9)
- moved C2 1.40 mm to (107.2, 112.3)
- moved R25 1.17 mm to (168.1, 72.6)
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Connections:
- C1 pad 1: BATT_MONITOR -> (no net)
- C3 pad 2: MOTOR_RESET -> Net-(C3-Pad2)
- R11 pad 1: SW -> Net-(R11-Pad1)
- R14 pad 1: IR_LED -> (no net)
- R3 pad 2: Net-(C2-Pad1) -> Net-(R3-Pad2)
- R4 pad 1: Net-(C2-Pad1) -> Net-(R3-Pad2)
- R5 pad 1: Net-(F1-Pad1) -> (no net)
- R6 pad 1: MOTOR_RESET -> Net-(C3-Pad2)
- R8 pad 1: +3V3 -> (no net)
- SW3 pad 1: SW -> Net-(R11-Pad1)
Routing:
- net SW: track 48.1 -> 9.36 mm
- net BATT_MONITOR: track 55.4 -> 28.2 mm
- net Net-(R22-Pad1): track 35.8 -> 61.9 mm
- net Net-(D3-Pad2): track 3.81 -> 27.4 mm
- net Net-(R17-Pad1): track 18.0 -> 40.5 mm
- net Net-(R19-Pad1): track 13.5 -> 35.6 mm
- net LCD_SCL: track 36.7 -> 58.5 mm, vias 0 -> 1
- net Net-(R18-Pad1): track 12.7 -> 33.0 mm
- net SWCLK: track 65.8 -> 47.6 mm
- net Net-(R21-Pad1): track 7.13 -> 24.4 mm
- net Net-(C2-Pad1): track 25.6 -> 9.11 mm
- net Net-(F1-Pad1): track 23.4 -> 7.18 mm
- net Net-(R20-Pad1): track 11.7 -> 27.8 mm
- net MOTOR_RESET: track 52.7 -> 37.7 mm
- net LCD_SDA: track 34.1 -> 48.9 mm
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Other:
- board text added: "Cheese Tutorial Boardv2"
- board text removed: "Cheese Tutorial Board"
