File: CheeseUnua.sch (KiCad schematic (older format))
At the start: 63 parts, among them J1 Jack-DC, J2 Battery, J3 Conn_01x05, J4 Conn_01x03, J5 Conn_01x06, J6 AE-AQM0802, J7 CN2, J8 CN1, Q1 2SJ681, Q2 2SK2796L, SW1 SW_SPDT, SW2 SW_SPST, SW3 SW_DPST_x2, U1 R-78E3.3-0.5, U2 SLA7073MPRT, U3 7SEGMENT_CA, U4 NJM2742D, U5 NJU7072D

Commit message: Step up to version 2
Parts:
- removed SW1: SW_SPDT, Pin_Headers:Pin_Header_Straight_1x03_Pitch2.54mm, symbol CheeseUnua-rescue:SW_SPDT-
- added JP1: Jumper_3_Bridged12, Pin_Headers:Pin_Header_Straight_1x03_Pitch2.54mm, symbol Jumper:Jumper_3_Bridged12
- J5: footprint Connectors_JST:JST_PH_B6B-PH-K_06x2.00mm_Straight -> Connectors_JST:JST_XH_S06B-XH-A_06x2.50mm_Angled
- R1, R10, R11, R12, R13, R14, R15, R16, R17, R18, R19, R2, R20, R21, R22, R23, R25, R26, R3, R4, R5, R6, R7, R8, R9: footprint Resistors_THT:R_Axial_DIN0204_L3.6mm_D1.6mm_P5.08mm_Horizontal -> Resistors_THT:R_Axial_DIN0204_L3.6mm_D1.6mm_P7.62mm_Horizontal
- R24: footprint Resistors_THT:R_Axial_DIN0204_L3.6mm_D1.6mm_P5.08mm_Horizontal -> Resistors_THT:R_Axial_DIN0207_L6.3mm_D2.5mm_P10.16mm_Horizontal
Connections:
- wire segments 95 -> 96
Other:
- moved on the sheet: J2
